Commit message: refactor + add link3, remove camera

File: acrobat_description/urdf/acrobat_gazebo.urdf.xacro (robot description, xacro)
@@ -1,66 +1,22 @@
 <?xml version="1.0"?>
 <robot>
-  <!-- Link1 -->
+  <gazebo>
+    <!-- ros_control plugin to actuate the acrobat joint -->
+    <plugin name="gazebo_ros_control" filename="libgazebo_ros_control.so" />
+    <!-- gazebo joint state publisher -->
+    <plugin name="gazebo_ros_joint_state_publisher" filename="libgazebo_ros_joint_state_publisher.so">
+      <jointName>joint1</jointName>
+      <updateRate>30.0</updateRate>
+    </plugin>
+  </gazebo>
+  <!-- Link colors -->
   <gazebo reference="link1">
     <material>Gazebo/DarkGrey</material>
   </gazebo>
-  <!-- Link2 -->
   <gazebo reference="link2">
-    <mu1>0.2</mu1>
-    <mu2>0.2</mu2>
-    <material>Gazebo/GreenTransparent</material>
+    <material>Gazebo/Green</material>
   </gazebo>
-  <!-- camera_link -->
-  <gazebo reference="camera_link">
-    <mu1>0.2</mu1>
-    <mu2>0.2</mu2>
-    <material>Gazebo/Grey</material>
-  </gazebo>
-  <!-- camera -->
-  <gazebo reference="camera_link">
-    <sensor type="camera" name="camera1">
-      <update_rate>30.0</update_rate>
-      <camera name="head">
-        <horizontal_fov>1.3962634</horizontal_fov>
-        <image>
-          <width>800</width>
-          <height>800</height>
-          <format>R8G8B8</format>
-        </image>
-        <clip>
-          <near>0.02</near>
-          <far>300</far>
-        </clip>
-        <noise>
-          <type>gaussian</type>
-          <!-- Noise is sampled independently per pixel on each frame.
-               That pixel's noise value is added to each of its color
-               channels, which at that point lie in the range [0,1]. -->
-          <mean>0.0</mean>
-          <stddev>0.007</stddev>
-        </noise>
-      </camera>
-      <plugin name="camera_controller" filename="libgazebo_ros_camera.so">
-        <alwaysOn>true</alwaysOn>
-        <updateRate>0.0</updateRate>
-        <cameraName>acrobat/camera1</cameraName>
-        <imageTopicName>image_raw</imageTopicName>
-        <cameraInfoTopicName>camera_info</cameraInfoTopicName>
-        <frameName>camera_link_optical</frameName>
-        <!-- setting hackBaseline to anything but 0.0 will cause a misalignment
-            between the gazebo sensor image and the frame it is supposed to
-            be attached to -->
-        <hackBaseline>0.0</hackBaseline>
-        <distortionK1>0.0</distortionK1>
-        <distortionK2>0.0</distortionK2>
-        <distortionK3>0.0</distortionK3>
-        <distortionT1>0.0</distortionT1>
-        <distortionT2>0.0</distortionT2>
-        <CxPrime>0</CxPrime>
-        <Cx>0.0</Cx>
-        <Cy>0.0</Cy>
-        <focalLength>0.0</focalLength>
-      </plugin>
-    </sensor>
+  <gazebo reference="link3">
+    <material>Gazebo/Orange</material>
   </gazebo>
 </robot>

File: acrobat_description/urdf/acrobat_robot.urdf.xacro (robot description, xacro)
@@ -1,140 +1,138 @@
 <?xml version="1.0"?>
-<!-- Revolute 1 joint manipulator -->
 <robot name="acrobat" xmlns:xacro="http://www.ros.org/wiki/xacro">
-  <!-- Constants for robot dimensions -->
-  <xacro:property name="PI" value="3.1415926535897931"/>
+  <!-- Robot properties -->
   <xacro:property name="mass" value="1" /> <!-- arbitrary value for mass -->
-  <xacro:property name="width" value="0.1" /> <!-- Square dimensions (widthxwidth) of beams -->
-  <xacro:property name="height1" value="2" /> <!-- Link 1 -->
-  <xacro:property name="height2" value="1" /> <!-- Link 2 -->
-  <xacro:property name="camera_link" value="0.05" /> <!-- Size of square 'camera' box -->
+  <xacro:property name="link_width" value="0.1" /> <!-- link square dimensions (link_widthxlink_width) -->
   <xacro:property name="axel_offset" value="0.05" /> <!-- Space btw top of beam and the each joint -->
+  <!-- link1 properties -->
+  <xacro:property name="link1_name" value="link1" />
+  <xacro:property name="link1_height" value="2" />
+  <!-- link2 properties -->
+  <xacro:property name="link2_name" value="link2" />
+  <xacro:property name="link2_height" value="1" />
+  <!-- link3 properties -->
+  <xacro:property name="link3_name" value="link3" />
+  <xacro:property name="link3_height" value="0.5" />
+  <!-- joint properties -->
+  <xacro:property name="joint_lower_limit" value="-3.1415" />
+  <xacro:property name="joint_upper_limit" value="3.1415" />
+  <xacro:property name="joint_effort" value="1000.0" />
+  <xacro:property name="joint_velocity" value="0.5" />
   <!-- Import Rviz colors -->
   <xacro:include filename="$(find acrobat_description)/urdf/materials.urdf.xacro" />
   <!-- Used for fixing robot to Gazebo 'base_link' -->
   <link name="world"/>
-  <joint name="fixed" type="fixed">
-    <parent link="world"/>
-    <child link="link1"/>
-  </joint>
-  <!-- Base Link -->
-  <link name="link1">
+  <!-- link1 -->
+  <link name="${link1_name}">
     <collision>
-      <origin xyz="0 0 ${height1/2}" rpy="0 0 0"/>
+      <origin xyz="0 0 ${link1_height/2}" rpy="0 0 0"/>
       <geometry>
-        <box size="${width} ${width} ${height1}"/>
+        <box size="${link_width} ${link_width} ${link1_height}"/>
       </geometry>
     </collision>
     <visual>
-      <origin xyz="0 0 ${height1/2}" rpy="0 0 0"/>
+      <origin xyz="0 0 ${link1_height/2}" rpy="0 0 0"/>
       <geometry>
-        <box size="${width} ${width} ${height1}"/>
+        <box size="${link_width} ${link_width} ${link1_height}"/>
       </geometry>
       <material name="black"/>
     </visual>
     <inertial>
-      <origin xyz="0 0 ${height1/2}" rpy="0 0 0"/>
+      <origin xyz="0 0 ${link1_height/2}" rpy="0 0 0"/>
       <mass value="${mass}"/>
       <inertia
-          ixx="${mass / 12.0 * (width*width + height1*height1)}" ixy="0.0" ixz="0.0"
-          iyy="${mass / 12.0 * (height1*height1 + width*width)}" iyz="0.0"
-          izz="${mass / 12.0 * (width*width + width*width)}"/>
+          ixx="${mass / 12.0 * (link_width*link_width + link1_height*link1_height)}" ixy="0.0" ixz="0.0"
+          iyy="${mass / 12.0 * (link1_height*link1_height + link_width*link_width)}" iyz="0.0"
+          izz="${mass / 12.0 * (link_width*link_width + link_width*link_width)}"/>
     </inertial>
   </link>
-  <joint name="joint1" type="continuous">
-    <parent link="link1"/>
-    <child link="link2"/>
-    <origin xyz="0 ${width} ${height1 - axel_offset}" rpy="0 0 0"/>
-    <axis xyz="0 1 0"/>
-    <dynamics damping="0.7"/>
+  <!-- joint0 -->
+  <joint name="fixed" type="fixed">
+    <parent link="world"/>
+    <child link="${link1_name}"/>
   </joint>
-  <!-- Acrobat green link -->
-  <link name="link2">
+  <!-- link2 -->
+  <link name="${link2_name}">
     <collision>
-      <origin xyz="0 0 ${height2/2 - axel_offset}" rpy="0 0 0"/>
+      <origin xyz="0 0 ${link2_height/2 - axel_offset}" rpy="0 0 0"/>
       <geometry>
-        <box size="${width} ${width} ${height2}"/>
+        <box size="${link_width} ${link_width} ${link2_height}"/>
       </geometry>
     </collision>
     <visual>
-      <origin xyz="0 0 ${height2/2 - axel_offset}" rpy="0 0 0"/>
+      <origin xyz="0 0 ${link2_height/2 - axel_offset}" rpy="0 0 0"/>
       <geometry>
-        <box size="${width} ${width} ${height2}"/>
+        <box size="${link_width} ${link_width} ${link2_height}"/>
       </geometry>
       <material name="green"/>
     </visual>
     <inertial>
-      <origin xyz="0 0 ${height2/2 - axel_offset}" rpy="0 0 0"/>
+      <origin xyz="0 0 ${link2_height/2 - axel_offset}" rpy="0 0 0"/>
       <mass value="${mass}"/>
       <inertia
-          ixx="${mass / 12.0 * (width*width + height2*height2)}" ixy="0.0" ixz="0.0"
-          iyy="${mass / 12.0 * (height2*height2 + width*width)}" iyz="0.0"
-          izz="${mass / 12.0 * (width*width + width*width)}"/>
+          ixx="${mass / 12.0 * (link_width*link_width + link2_height*link2_height)}" ixy="0.0" ixz="0.0"
+          iyy="${mass / 12.0 * (link2_height*link2_height + link_width*link_width)}" iyz="0.0"
+          izz="${mass / 12.0 * (link_width*link_width + link_width*link_width)}"/>
     </inertial>
   </link>
-  <joint name="camera_joint" type="fixed">
-    <axis xyz="0 1 0" />
-    <origin xyz="${camera_link} 0 ${height2 - axel_offset*2}" rpy="0 0 0"/>
-    <parent link="link2"/>
-    <child link="camera_link"/>
+  <!-- joint1 -->
+  <joint name="${link1_name}_to_${link2_name}_joint" type="revolute">
+    <parent link="${link1_name}"/>
+    <child link="${link2_name}"/>
+    <origin xyz="0 ${link_width} ${link1_height - axel_offset}" rpy="0 0 0"/>
+    <axis xyz="0 1 0"/>
+    <dynamics damping="0.7"/>
+    <limit effort="1000.0" lower="${joint_lower_limit}" upper="${joint_upper_limit}" velocity="0.5"/>
   </joint>
-  <!-- dummy link to get a tf at the end of link2 -->
-  <link name="link3" />
-  <!-- dummy fixed joint to get a tf at the end of link2 (for reward calculation purposes -> learning stuff) -->
-  <joint name="link3_joint" type="fixed">
-    <axis xyz="0 0 1" />
-    <origin xyz="0 0 ${height2}" rpy="0 0 0"/>
-    <parent link="link2"/>
-    <child link="link3"/>
-  </joint>
-  <!-- if link3 matches exactly with this one, then reward of the acrobat is maximum -->
-  <link name="goal_link" />
-  <joint name="goal_link_joint" type="fixed">
-    <axis xyz="0 0 1" />
-    <origin xyz="0 ${width} ${height1 + height2 - axel_offset}" rpy="0 0 0"/>
-    <parent link="link1"/>
-    <child link="goal_link"/>
-  </joint>
-  <!-- Camera -->
-  <link name="camera_link">
+  <!-- link3 -->
+  <link name="${link3_name}">
     <collision>
-      <origin xyz="0 0 0" rpy="0 0 0"/>
+      <origin xyz="0 0 ${link3_height/2 - axel_offset}" rpy="0 0 0"/>
       <geometry>
-        <box size="${camera_link} ${camera_link} ${camera_link}"/>
+        <box size="${link_width} ${link_width} ${link3_height}"/>
       </geometry>
     </collision>
     <visual>
-      <origin xyz="0 0 0" rpy="0 0 0"/>
+      <origin xyz="0 0 ${link3_height/2 - axel_offset}" rpy="0 0 0"/>
       <geometry>
-        <box size="${camera_link} ${camera_link} ${camera_link}"/>
+        <box size="${link_width} ${link_width} ${link3_height}"/>
       </geometry>
-      <material name="grey"/>
+      <material name="green"/>
     </visual>
     <inertial>
-      <mass value="1e-5" />
-      <origin xyz="0 0 0" rpy="0 0 0"/>
-      <inertia ixx="1e-6" ixy="0" ixz="0" iyy="1e-6" iyz="0" izz="1e-6" />
+      <origin xyz="0 0 ${link3_height/2 - axel_offset}" rpy="0 0 0"/>
+      <mass value="${mass}"/>
+      <inertia
+          ixx="${mass / 12.0 * (link_width*link_width + link3_height*link3_height)}" ixy="0.0" ixz="0.0"
+          iyy="${mass / 12.0 * (link3_height*link3_height + link_width*link_width)}" iyz="0.0"
+          izz="${mass / 12.0 * (link_width*link_width + link_width*link_width)}"/>
     </inertial>
   </link>
-  <!-- generate an optical frame http://www.ros.org/reps/rep-0103.html#suffix-frames
-      so that ros and opencv can operate on the camera frame correctly -->
-  <joint name="camera_optical_joint" type="fixed">
-    <!-- these values have to be these values otherwise the gazebo camera image
-        won't be aligned properly with the frame it is supposedly originating from -->
-    <origin xyz="0 0 0" rpy="${-pi/2} 0 ${-pi/2}"/>
-    <parent link="camera_link"/>
-    <child link="camera_link_optical"/>
+  <!-- joint2 -->
+  <joint name="${link2_name}_to_${link3_name}_joint" type="revolute">
+    <parent link="${link2_name}"/>
+    <child link="${link3_name}"/>
+    <origin xyz="0 ${link_width} ${link2_height - axel_offset}" rpy="0 0 0"/>
+    <axis xyz="0 1 0"/>
+    <dynamics damping="0.7"/>
+    <limit effort="${joint_effort}" lower="${joint_lower_limit}" upper="${joint_upper_limit}" velocity="${joint_velocity}"/>
   </joint>
-  <link name="camera_link_optical">
-  </link>
-  <transmission name="tran1">
-    <type>transmission_interface/SimpleTransmission</type>
-    <joint name="joint1">
-      <hardwareInterface>hardware_interface/EffortJointInterface</hardwareInterface>
-    </joint>
-    <actuator name="motor1">
-      <hardwareInterface>hardware_interface/EffortJointInterface</hardwareInterface>
-      <mechanicalReduction>1</mechanicalReduction>
-    </actuator>
-  </transmission>
+  <!-- arm transmission macro (needed to actuate joints in gazebo simulator via ROS control) -->
+  <xacro:macro name="arm_transmission_macro" params="joint_name">
+    <transmission name="${joint_name}_trans">
+      <type>transmission_interface/SimpleTransmission</type>
+      <joint name="${joint_name}">
+        <hardwareInterface>hardware_interface/EffortJointInterface</hardwareInterface>
+      </joint>
+      <actuator name="${joint_name}_actuator">
+        <mechanicalReduction>1</mechanicalReduction>
+      </actuator>
+    </transmission>
+  </xacro:macro>
+  <!-- joint1 -->
+  <xacro:arm_transmission_macro joint_name="${link1_name}_to_${link2_name}_joint" />
+  <!-- joint2 -->
+  <xacro:arm_transmission_macro joint_name="${link2_name}_to_${link3_name}_joint" />
+  <!-- gazebo related tags -->
+  <xacro:include filename="$(find acrobat_description)/urdf/acrobat_gazebo.urdf.xacro" />
 </robot>

Commit message: reduce to 2 links and fix robot to 2D environment

File: acrobat_description/urdf/acrobat_gazebo.urdf.xacro (robot description, xacro)
@@ -17,6 +17,3 @@
     <material>Gazebo/Green</material>
   </gazebo>
-  <gazebo reference="link3">
-    <material>Gazebo/Orange</material>
-  </gazebo>
 </robot>

File: acrobat_description/urdf/acrobat_robot.urdf.xacro (robot description, xacro)
@@ -3,23 +3,18 @@
   <!-- Math properties -->
   <xacro:property name="PI" value="3.141592653589793" />
-  <!-- Robot properties -->
-  <xacro:property name="mass" value="1" /> <!-- arbitrary value for mass -->
+  <!-- link properties -->
+  <xacro:property name="link_mass" value="1" /> <!-- arbitrary value for mass -->
   <xacro:property name="link_width" value="0.1" /> <!-- link square dimensions (link_widthxlink_width) -->
-  <xacro:property name="axel_offset" value="0.05" /> <!-- Space btw top of beam and the each joint -->
   <!-- link1 properties -->
   <xacro:property name="link1_name" value="link1" />
-  <xacro:property name="link1_height" value="2" />
+  <xacro:property name="link1_height" value="3.0" />
   <xacro:property name="link1_color" value="grey" />
   <!-- link2 properties -->
   <xacro:property name="link2_name" value="link2" />
-  <xacro:property name="link2_height" value="1" />
+  <xacro:property name="link2_height" value="2.0" />
   <xacro:property name="link2_color" value="green" />
-  <!-- link3 properties -->
-  <xacro:property name="link3_name" value="link3" />
-  <xacro:property name="link3_height" value="0.5" />
-  <xacro:property name="link3_color" value="orange" />
   <!-- joint properties -->
-  <xacro:property name="joint_lower_limit" value="${-PI/2.0}" />
-  <xacro:property name="joint_upper_limit" value="${PI/2.0}" />
+  <xacro:property name="joint_lower_limit" value="${-PI / 2.0}" />
+  <xacro:property name="joint_upper_limit" value="${PI / 2.0}" />
   <xacro:property name="joint_effort" value="1000.0" />
   <xacro:property name="joint_velocity" value="0.5" />
@@ -29,25 +24,25 @@
   <xacro:macro name="link_macro" params="link_name link_height link_color">
     <link name="${link_name}">
-        <collision>
-        <origin xyz="0 0 ${link_height/2}" rpy="0 0 0"/>
+      <visual>
+        <origin xyz="${link_height/2} 0 0" rpy="0 0 0"/>
         <geometry>
-            <box size="${link_width} ${link_width} ${link_height}"/>
-        </geometry>
-        </collision>
-        <visual>
-        <origin xyz="0 0 ${link_height/2}" rpy="0 0 0"/>
-        <geometry>
-            <box size="${link_width} ${link_width} ${link_height}"/>
+          <box size="${link_height} ${link_width} ${link_width}"/>
         </geometry>
         <material name="${link_color}"/>
-        </visual>
-        <inertial>
-        <origin xyz="0 0 ${link_height/2}" rpy="0 0 0"/>
-        <mass value="${mass}"/>
+      </visual>
+      <collision>
+        <origin xyz="${link_height/2} 0 0" rpy="0 0 0"/>
+        <geometry>
+          <box size="${link_height} ${link_width} ${link_width}"/>
+        </geometry>
+      </collision>
+      <inertial>
+        <origin xyz="${link_height/2} 0 0" rpy="0 0 0"/>
+        <mass value="${link_mass}"/>
         <inertia
-            ixx="${mass / 12.0 * (link_width*link_width + link_height*link_height)}" ixy="0.0" ixz="0.0"
-            iyy="${mass / 12.0 * (link_height*link_height + link_width*link_width)}" iyz="0.0"
-            izz="${mass / 12.0 * (link_width*link_width + link_width*link_width)}"/>
-        </inertial>
+            ixx="${link_mass / 12.0 * (link_width*link_width + link_height*link_height)}" ixy="0.0" ixz="0.0"
+            iyy="${link_mass / 12.0 * (link_height*link_height + link_width*link_width)}" iyz="0.0"
+            izz="${link_mass / 12.0 * (link_width*link_width + link_width*link_width)}"/>
+      </inertial>
     </link>
   </xacro:macro>
@@ -55,10 +50,10 @@
   <xacro:macro name="joint_macro" params="joint_name parent_link child_link parent_link_height">
     <joint name="${parent_link}_to_${child_link}_joint" type="revolute">
-        <parent link="${parent_link}"/>
-        <child link="${child_link}"/>
-        <origin xyz="0 ${link_width} ${parent_link_height - axel_offset}" rpy="0 0 0"/>
-        <axis xyz="0 1 0"/>
-        <dynamics damping="0.7"/>
-        <limit effort="${joint_effort}" lower="${joint_lower_limit}" upper="${joint_upper_limit}" velocity="${joint_velocity}"/>
+      <parent link="${parent_link}"/>
+      <child link="${child_link}"/>
+      <origin xyz="${parent_link_height} 0 ${parent_link_height - link_width / 2.0}" rpy="0 0 0"/>
+      <axis xyz="0 0 1"/>
+      <dynamics damping="0.7"/>
+      <limit effort="${joint_effort}" lower="${joint_lower_limit}" upper="${joint_upper_limit}" velocity="${joint_velocity}"/>
     </joint>
     <transmission name="${joint_name}_trans">
@@ -72,19 +67,19 @@
     </transmission>
   </xacro:macro>
-  <!-- link0 -->
+  <!-- link 0, 1 -->
   <link name="world"/>
-  <!-- links 1, 2, 3 -->
+  <link name="dummy_link"/>
+  <!-- links 2, 3 -->
   <xacro:link_macro link_name="${link1_name}" link_height="${link1_height}" link_color="${link1_color}" />
   <xacro:link_macro link_name="${link2_name}" link_height="${link2_height}" link_color="${link2_color}" />
-  <xacro:link_macro link_name="${link3_name}" link_height="${link3_height}" link_color="${link3_color}" />
   <!-- joint0 -->
   <joint name="fixed" type="fixed">
     <parent link="world"/>
-    <child link="${link1_name}"/>
-    <origin xyz="0 0 0" rpy="${-PI/2.0} 0 0"/>
+    <child link="dummy_link"/>
+    <origin xyz="0 0 0" rpy="0 0 0"/>
   </joint>
   <!-- joints 1, 2 -->
-  <xacro:joint_macro joint_name="joint1" parent_link="${link1_name}" child_link="${link2_name}" parent_link_height="${link1_height}" />
-  <xacro:joint_macro joint_name="joint2" parent_link="${link2_name}" child_link="${link3_name}" parent_link_height="${link2_height}" />
+  <xacro:joint_macro joint_name="joint1" parent_link="dummy_link" child_link="${link1_name}" parent_link_height="0" />
+  <xacro:joint_macro joint_name="joint2" parent_link="${link1_name}" child_link="${link2_name}" parent_link_height="${link1_height}" />
   <!-- gazebo related tags -->
   <xacro:include filename="$(find acrobat_description)/urdf/acrobat_gazebo.urdf.xacro" />

Commit message: first working version

File: acrobat_description/urdf/acrobat_gazebo.urdf.xacro (robot description, xacro)
@@ -1,12 +1,7 @@
 <?xml version="1.0"?>
 <robot>
+  <!-- ros_control plugin to actuate the acrobat joint -->
   <gazebo>
-    <!-- ros_control plugin to actuate the acrobat joint -->
     <plugin name="gazebo_ros_control" filename="libgazebo_ros_control.so" />
-    <!-- gazebo joint state publisher -->
-    <plugin name="gazebo_ros_joint_state_publisher" filename="libgazebo_ros_joint_state_publisher.so">
-      <jointName>joint1</jointName>
-      <updateRate>30.0</updateRate>
-    </plugin>
   </gazebo>
   <!-- Link colors -->

File: acrobat_description/urdf/acrobat_robot.urdf.xacro (robot description, xacro)
@@ -4,5 +4,5 @@
   <xacro:property name="PI" value="3.141592653589793" />
   <!-- link properties -->
-  <xacro:property name="link_mass" value="1" /> <!-- arbitrary value for mass -->
+  <xacro:property name="link_mass" value="0.1" /> <!-- arbitrary value for mass -->
   <xacro:property name="link_width" value="0.1" /> <!-- link square dimensions (link_widthxlink_width) -->
   <!-- link1 properties -->
@@ -49,8 +49,8 @@
   <!-- joint macro -->
   <xacro:macro name="joint_macro" params="joint_name parent_link child_link parent_link_height">
-    <joint name="${parent_link}_to_${child_link}_joint" type="revolute">
+    <joint name="${joint_name}" type="revolute">
       <parent link="${parent_link}"/>
       <child link="${child_link}"/>
-      <origin xyz="${parent_link_height} 0 ${parent_link_height - link_width / 2.0}" rpy="0 0 0"/>
+      <origin xyz="${parent_link_height} 0 ${link_width}" rpy="0 0 0"/>
       <axis xyz="0 0 1"/>
       <dynamics damping="0.7"/>
@@ -69,10 +69,19 @@
   <!-- link 0, 1 -->
   <link name="world"/>
-  <link name="dummy_link"/>
+  <link name="dummy_link">
+    <inertial>
+      <origin xyz="0 0 0" rpy="0 0 0"/>
+      <mass value="${link_mass}"/>
+      <inertia
+        ixx="0.001" ixy="0.0" ixz="0.0"
+        iyy="0.001" iyz="0.0"
+        izz="0.001"/>
+    </inertial>
+  </link>
   <!-- links 2, 3 -->
   <xacro:link_macro link_name="${link1_name}" link_height="${link1_height}" link_color="${link1_color}" />
   <xacro:link_macro link_name="${link2_name}" link_height="${link2_height}" link_color="${link2_color}" />
   <!-- joint0 -->
-  <joint name="fixed" type="fixed">
+  <joint name="joint0" type="fixed">
     <parent link="world"/>
     <child link="dummy_link"/>
