Commit message: convert urdf into macro

File: acrobat_description/urdf/acrobat_robot.urdf.xacro (robot description, xacro)
@@ -1,4 +1,6 @@
 <?xml version="1.0"?>
 <robot name="acrobat" xmlns:xacro="http://www.ros.org/wiki/xacro">
+  <!-- Math properties -->
+  <xacro:property name="PI" value="3.141592653589793" />
   <!-- Robot properties -->
   <xacro:property name="mass" value="1" /> <!-- arbitrary value for mass -->
@@ -8,116 +10,56 @@
   <xacro:property name="link1_name" value="link1" />
   <xacro:property name="link1_height" value="2" />
+  <xacro:property name="link1_color" value="grey" />
   <!-- link2 properties -->
   <xacro:property name="link2_name" value="link2" />
   <xacro:property name="link2_height" value="1" />
+  <xacro:property name="link2_color" value="green" />
   <!-- link3 properties -->
   <xacro:property name="link3_name" value="link3" />
   <xacro:property name="link3_height" value="0.5" />
+  <xacro:property name="link3_color" value="orange" />
   <!-- joint properties -->
-  <xacro:property name="joint_lower_limit" value="-3.1415" />
-  <xacro:property name="joint_upper_limit" value="3.1415" />
+  <xacro:property name="joint_lower_limit" value="${-PI/2.0}" />
+  <xacro:property name="joint_upper_limit" value="${PI/2.0}" />
   <xacro:property name="joint_effort" value="1000.0" />
   <xacro:property name="joint_velocity" value="0.5" />
   <!-- Import Rviz colors -->
   <xacro:include filename="$(find acrobat_description)/urdf/materials.urdf.xacro" />
-  <!-- Used for fixing robot to Gazebo 'base_link' -->
-  <link name="world"/>
-  <!-- link1 -->
-  <link name="${link1_name}">
-    <collision>
-      <origin xyz="0 0 ${link1_height/2}" rpy="0 0 0"/>
-      <geometry>
-        <box size="${link_width} ${link_width} ${link1_height}"/>
-      </geometry>
-    </collision>
-    <visual>
-      <origin xyz="0 0 ${link1_height/2}" rpy="0 0 0"/>
-      <geometry>
-        <box size="${link_width} ${link_width} ${link1_height}"/>
-      </geometry>
-      <material name="black"/>
-    </visual>
-    <inertial>
-      <origin xyz="0 0 ${link1_height/2}" rpy="0 0 0"/>
-      <mass value="${mass}"/>
-      <inertia
-          ixx="${mass / 12.0 * (link_width*link_width + link1_height*link1_height)}" ixy="0.0" ixz="0.0"
-          iyy="${mass / 12.0 * (link1_height*link1_height + link_width*link_width)}" iyz="0.0"
-          izz="${mass / 12.0 * (link_width*link_width + link_width*link_width)}"/>
-    </inertial>
-  </link>
-  <!-- joint0 -->
-  <joint name="fixed" type="fixed">
-    <parent link="world"/>
-    <child link="${link1_name}"/>
-  </joint>
-  <!-- link2 -->
-  <link name="${link2_name}">
-    <collision>
-      <origin xyz="0 0 ${link2_height/2 - axel_offset}" rpy="0 0 0"/>
-      <geometry>
-        <box size="${link_width} ${link_width} ${link2_height}"/>
-      </geometry>
-    </collision>
-    <visual>
-      <origin xyz="0 0 ${link2_height/2 - axel_offset}" rpy="0 0 0"/>
-      <geometry>
-        <box size="${link_width} ${link_width} ${link2_height}"/>
-      </geometry>
-      <material name="green"/>
-    </visual>
-    <inertial>
-      <origin xyz="0 0 ${link2_height/2 - axel_offset}" rpy="0 0 0"/>
-      <mass value="${mass}"/>
-      <inertia
-          ixx="${mass / 12.0 * (link_width*link_width + link2_height*link2_height)}" ixy="0.0" ixz="0.0"
-          iyy="${mass / 12.0 * (link2_height*link2_height + link_width*link_width)}" iyz="0.0"
-          izz="${mass / 12.0 * (link_width*link_width + link_width*link_width)}"/>
-    </inertial>
-  </link>
-  <!-- joint1 -->
-  <joint name="${link1_name}_to_${link2_name}_joint" type="revolute">
-    <parent link="${link1_name}"/>
-    <child link="${link2_name}"/>
-    <origin xyz="0 ${link_width} ${link1_height - axel_offset}" rpy="0 0 0"/>
-    <axis xyz="0 1 0"/>
-    <dynamics damping="0.7"/>
-    <limit effort="1000.0" lower="${joint_lower_limit}" upper="${joint_upper_limit}" velocity="0.5"/>
-  </joint>
-  <!-- link3 -->
-  <link name="${link3_name}">
-    <collision>
-      <origin xyz="0 0 ${link3_height/2 - axel_offset}" rpy="0 0 0"/>
-      <geometry>
-        <box size="${link_width} ${link_width} ${link3_height}"/>
-      </geometry>
-    </collision>
-    <visual>
-      <origin xyz="0 0 ${link3_height/2 - axel_offset}" rpy="0 0 0"/>
-      <geometry>
-        <box size="${link_width} ${link_width} ${link3_height}"/>
-      </geometry>
-      <material name="green"/>
-    </visual>
-    <inertial>
-      <origin xyz="0 0 ${link3_height/2 - axel_offset}" rpy="0 0 0"/>
-      <mass value="${mass}"/>
-      <inertia
-          ixx="${mass / 12.0 * (link_width*link_width + link3_height*link3_height)}" ixy="0.0" ixz="0.0"
-          iyy="${mass / 12.0 * (link3_height*link3_height + link_width*link_width)}" iyz="0.0"
-          izz="${mass / 12.0 * (link_width*link_width + link_width*link_width)}"/>
-    </inertial>
-  </link>
-  <!-- joint2 -->
-  <joint name="${link2_name}_to_${link3_name}_joint" type="revolute">
-    <parent link="${link2_name}"/>
-    <child link="${link3_name}"/>
-    <origin xyz="0 ${link_width} ${link2_height - axel_offset}" rpy="0 0 0"/>
-    <axis xyz="0 1 0"/>
-    <dynamics damping="0.7"/>
-    <limit effort="${joint_effort}" lower="${joint_lower_limit}" upper="${joint_upper_limit}" velocity="${joint_velocity}"/>
-  </joint>
-  <!-- arm transmission macro (needed to actuate joints in gazebo simulator via ROS control) -->
-  <xacro:macro name="arm_transmission_macro" params="joint_name">
+  <!-- link macro -->
+  <xacro:macro name="link_macro" params="link_name link_height link_color">
+    <link name="${link_name}">
+        <collision>
+        <origin xyz="0 0 ${link_height/2}" rpy="0 0 0"/>
+        <geometry>
+            <box size="${link_width} ${link_width} ${link_height}"/>
+        </geometry>
+        </collision>
+        <visual>
+        <origin xyz="0 0 ${link_height/2}" rpy="0 0 0"/>
+        <geometry>
+            <box size="${link_width} ${link_width} ${link_height}"/>
+        </geometry>
+        <material name="${link_color}"/>
+        </visual>
+        <inertial>
+        <origin xyz="0 0 ${link_height/2}" rpy="0 0 0"/>
+        <mass value="${mass}"/>
+        <inertia
+            ixx="${mass / 12.0 * (link_width*link_width + link_height*link_height)}" ixy="0.0" ixz="0.0"
+            iyy="${mass / 12.0 * (link_height*link_height + link_width*link_width)}" iyz="0.0"
+            izz="${mass / 12.0 * (link_width*link_width + link_width*link_width)}"/>
+        </inertial>
+    </link>
+  </xacro:macro>
+  <!-- joint macro -->
+  <xacro:macro name="joint_macro" params="joint_name parent_link child_link parent_link_height">
+    <joint name="${parent_link}_to_${child_link}_joint" type="revolute">
+        <parent link="${parent_link}"/>
+        <child link="${child_link}"/>
+        <origin xyz="0 ${link_width} ${parent_link_height - axel_offset}" rpy="0 0 0"/>
+        <axis xyz="0 1 0"/>
+        <dynamics damping="0.7"/>
+        <limit effort="${joint_effort}" lower="${joint_lower_limit}" upper="${joint_upper_limit}" velocity="${joint_velocity}"/>
+    </joint>
     <transmission name="${joint_name}_trans">
       <type>transmission_interface/SimpleTransmission</type>
@@ -130,8 +72,19 @@
     </transmission>
   </xacro:macro>
-  <!-- joint1 -->
-  <xacro:arm_transmission_macro joint_name="${link1_name}_to_${link2_name}_joint" />
-  <!-- joint2 -->
-  <xacro:arm_transmission_macro joint_name="${link2_name}_to_${link3_name}_joint" />
+  <!-- link0 -->
+  <link name="world"/>
+  <!-- links 1, 2, 3 -->
+  <xacro:link_macro link_name="${link1_name}" link_height="${link1_height}" link_color="${link1_color}" />
+  <xacro:link_macro link_name="${link2_name}" link_height="${link2_height}" link_color="${link2_color}" />
+  <xacro:link_macro link_name="${link3_name}" link_height="${link3_height}" link_color="${link3_color}" />
+  <!-- joint0 -->
+  <joint name="fixed" type="fixed">
+    <parent link="world"/>
+    <child link="${link1_name}"/>
+    <origin xyz="0 0 0" rpy="${-PI/2.0} 0 0"/>
+  </joint>
+  <!-- joints 1, 2 -->
+  <xacro:joint_macro joint_name="joint1" parent_link="${link1_name}" child_link="${link2_name}" parent_link_height="${link1_height}" />
+  <xacro:joint_macro joint_name="joint2" parent_link="${link2_name}" child_link="${link3_name}" parent_link_height="${link2_height}" />
   <!-- gazebo related tags -->
   <xacro:include filename="$(find acrobat_description)/urdf/acrobat_gazebo.urdf.xacro" />

Commit message: fix inertia, camera gazebo default pose, add arm pose c

File: acrobat_description/urdf/acrobat_robot.urdf.xacro (robot description, xacro)
@@ -38,5 +38,5 @@
       </collision>
       <inertial>
-        <origin xyz="${link_height/2} 0 0" rpy="0 0 0"/>
+        <origin xyz="${link_height/2} 0 0" rpy="0 ${PI/2.0} 0"/>
         <mass value="${link_mass}"/>
         <inertia

Commit message: various fixes to urdf model

File: acrobat_description/urdf/acrobat_robot.urdf.xacro (robot description, xacro)
@@ -3,22 +3,37 @@
   <!-- Math properties -->
   <xacro:property name="PI" value="3.141592653589793" />
-  <!-- link properties -->
+  <!-- common link properties -->
   <xacro:property name="link_mass" value="0.1" /> <!-- arbitrary value for mass -->
   <xacro:property name="link_width" value="0.1" /> <!-- link square dimensions (link_widthxlink_width) -->
   <!-- link1 properties -->
   <xacro:property name="link1_name" value="link1" />
-  <xacro:property name="link1_height" value="3.0" />
+  <xacro:property name="link1_height" value="${link_width}" />
   <xacro:property name="link1_color" value="grey" />
   <!-- link2 properties -->
   <xacro:property name="link2_name" value="link2" />
-  <xacro:property name="link2_height" value="2.0" />
+  <xacro:property name="link2_height" value="3.0" />
   <xacro:property name="link2_color" value="green" />
-  <!-- joint properties -->
+  <!-- link3 properties -->
+  <xacro:property name="link3_name" value="link3" />
+  <xacro:property name="link3_height" value="2.0" />
+  <xacro:property name="link3_color" value="orange" />
+  <!-- common joint properties -->
   <xacro:property name="joint_lower_limit" value="${-PI / 2.0}" />
   <xacro:property name="joint_upper_limit" value="${PI / 2.0}" />
-  <xacro:property name="joint_effort" value="1000.0" />
-  <xacro:property name="joint_velocity" value="0.5" />
+  <xacro:property name="joint_effort" value="100.0" />
+  <xacro:property name="joint_velocity" value="100.0" />
+  <xacro:property name="joint_damping" value="0.7" />
   <!-- Import Rviz colors -->
   <xacro:include filename="$(find acrobat_description)/urdf/materials.urdf.xacro" />
+  <!-- inertia macro -->
+  <xacro:macro name="box_inertial_with_origin" params="x y z mass *origin">
+    <inertial>
+      <mass value="${mass}" />
+      <xacro:insert_block name="origin" />
+      <inertia ixx="${0.0833333 * mass * (y*y + z*z)}" ixy="0.0" ixz="0.0"
+        iyy="${0.0833333 * mass * (x*x + z*z)}" iyz="0.0"
+        izz="${0.0833333 * mass * (x*x + y*y)}" />
+    </inertial>
+  </xacro:macro>
   <!-- link macro -->
   <xacro:macro name="link_macro" params="link_name link_height link_color">
@@ -37,22 +52,18 @@
         </geometry>
       </collision>
-      <inertial>
-        <origin xyz="${link_height/2} 0 0" rpy="0 ${PI/2.0} 0"/>
-        <mass value="${link_mass}"/>
-        <inertia
-            ixx="${link_mass / 12.0 * (link_width*link_width + link_height*link_height)}" ixy="0.0" ixz="0.0"
-            iyy="${link_mass / 12.0 * (link_height*link_height + link_width*link_width)}" iyz="0.0"
-            izz="${link_mass / 12.0 * (link_width*link_width + link_width*link_width)}"/>
-      </inertial>
+      <!-- use macro to compute inertia-->
+      <xacro:box_inertial_with_origin x="${link_height}" y="${link_width}" z="${link_width}" mass="${link_mass}" >
+        <origin xyz="${link_height/2} 0 0" rpy="0 0 0" />
+      </xacro:box_inertial_with_origin>
     </link>
   </xacro:macro>
   <!-- joint macro -->
-  <xacro:macro name="joint_macro" params="joint_name parent_link child_link parent_link_height">
+  <xacro:macro name="joint_macro" params="joint_name parent_link child_link *origin">
     <joint name="${joint_name}" type="revolute">
+      <xacro:insert_block name="origin" />
       <parent link="${parent_link}"/>
       <child link="${child_link}"/>
-      <origin xyz="${parent_link_height} 0 ${link_width}" rpy="0 0 0"/>
       <axis xyz="0 0 1"/>
-      <dynamics damping="0.7"/>
+      <dynamics damping="${joint_damping}"/>
       <limit effort="${joint_effort}" lower="${joint_lower_limit}" upper="${joint_upper_limit}" velocity="${joint_velocity}"/>
     </joint>
@@ -67,28 +78,23 @@
     </transmission>
   </xacro:macro>
-  <!-- link 0, 1 -->
+  <!-- link 0 -->
   <link name="world"/>
-  <link name="dummy_link">
-    <inertial>
-      <origin xyz="0 0 0" rpy="0 0 0"/>
-      <mass value="${link_mass}"/>
-      <inertia
-        ixx="0.001" ixy="0.0" ixz="0.0"
-        iyy="0.001" iyz="0.0"
-        izz="0.001"/>
-    </inertial>
-  </link>
-  <!-- links 2, 3 -->
+  <!-- links 1, 2, 3 -->
   <xacro:link_macro link_name="${link1_name}" link_height="${link1_height}" link_color="${link1_color}" />
   <xacro:link_macro link_name="${link2_name}" link_height="${link2_height}" link_color="${link2_color}" />
+  <xacro:link_macro link_name="${link3_name}" link_height="${link3_height}" link_color="${link3_color}" />
   <!-- joint0 -->
   <joint name="joint0" type="fixed">
     <parent link="world"/>
-    <child link="dummy_link"/>
+    <child link="${link1_name}"/>
     <origin xyz="0 0 0" rpy="0 0 0"/>
   </joint>
   <!-- joints 1, 2 -->
-  <xacro:joint_macro joint_name="joint1" parent_link="dummy_link" child_link="${link1_name}" parent_link_height="0" />
-  <xacro:joint_macro joint_name="joint2" parent_link="${link1_name}" child_link="${link2_name}" parent_link_height="${link1_height}" />
+  <xacro:joint_macro joint_name="joint1" parent_link="${link1_name}" child_link="${link2_name}" >
+    <origin xyz="0 0 ${link_width}" rpy="0 0 0"/>
+  </xacro:joint_macro>
+  <xacro:joint_macro joint_name="joint2" parent_link="${link2_name}" child_link="${link3_name}" >
+    <origin xyz="${link2_height} 0 ${link_width}" rpy="0 0 0"/>
+  </xacro:joint_macro>
   <!-- gazebo related tags -->
   <xacro:include filename="$(find acrobat_description)/urdf/acrobat_gazebo.urdf.xacro" />

Commit message: switch to vel control interface and tune pid

File: acrobat_description/urdf/acrobat_robot.urdf.xacro (robot description, xacro)
@@ -22,6 +22,5 @@
   <xacro:property name="joint_upper_limit" value="${PI / 2.0}" />
   <xacro:property name="joint_effort" value="100.0" />
-  <xacro:property name="joint_velocity" value="100.0" />
-  <xacro:property name="joint_damping" value="0.7" />
+  <xacro:property name="joint_velocity" value="1.0" />
   <!-- Import Rviz colors -->
   <xacro:include filename="$(find acrobat_description)/urdf/materials.urdf.xacro" />
@@ -65,5 +64,5 @@
       <child link="${child_link}"/>
       <axis xyz="0 0 1"/>
-      <dynamics damping="${joint_damping}"/>
+      <!--<dynamics damping="10.0" friction="10.0"/>-->
       <limit effort="${joint_effort}" lower="${joint_lower_limit}" upper="${joint_upper_limit}" velocity="${joint_velocity}"/>
     </joint>
@@ -71,5 +70,5 @@
       <type>transmission_interface/SimpleTransmission</type>
       <joint name="${joint_name}">
-        <hardwareInterface>hardware_interface/EffortJointInterface</hardwareInterface>
+        <hardwareInterface>hardware_interface/VelocityJointInterface</hardwareInterface>
       </joint>
       <actuator name="${joint_name}_actuator">

Commit message: resolve jittering problem, was touching with the ground, with wrong inertia and was having bad tuning on the controller

File: acrobat_description/urdf/acrobat_robot.urdf.xacro (robot description, xacro)
@@ -52,6 +52,6 @@
       </collision>
       <!-- use macro to compute inertia-->
-      <xacro:box_inertial_with_origin x="${link_height}" y="${link_width}" z="${link_width}" mass="${link_mass}" >
-        <origin xyz="${link_height/2} 0 0" rpy="0 0 0" />
+      <xacro:box_inertial_with_origin x="${link_width}" y="${link_width}" z="${link_width}" mass="${link_mass}" >
+        <origin xyz="0 0 0" rpy="0 0 0" />
       </xacro:box_inertial_with_origin>
     </link>
@@ -87,5 +87,5 @@
     <parent link="world"/>
     <child link="${link1_name}"/>
-    <origin xyz="0 0 0" rpy="0 0 0"/>
+    <origin xyz="0 0 0.5" rpy="0 0 0"/>
   </joint>
   <!-- joints 1, 2 -->
